File: board/Stm32CanBridge.kicad_pcb (KiCad board)
At the start: 2 copper layers, 43.2 x 35.6 mm, 20 parts, among them J1 DB9, P1 USB_B, P2 CONN_01X03, U1 LM1117-3.3, U2 MCP2562-E/SN, U3 STM32F042C4Tx

Commit message: edit silk
Other:
- board text added: "STM32 CAN <=> USB 15 Dec 2016"
- board text removed: "15 Dec 2016"
- board text removed: "STM32 CAN <=> USB"
Changed lines of the file:
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@@
     (area 137.084999 72.314999 180.415001 108.025001)
     (thickness 1.6)
-    (drawings 11)
+    (drawings 10)
     (tracks 143)
     (zones 0)
@@
     )
   )
-  (gr_text "Matthew Kennedy\nmck1117@github" (at 161.29 81.28 360) (layer B.SilkS)
+  (gr_text "Matthew Kennedy\nmck1117@github" (at 161.29 81.28) (layer B.SilkS)
     (effects (font (size 1 1) (thickness 0.1)) (justify mirror))
   )
-  (gr_text "15 Dec 2016" (at 172.72 90.17 270) (layer B.SilkS)
+  (gr_text "STM32 CAN <=> USB\n15 Dec 2016" (at 173.99 90.17 270) (layer B.SilkS)
     (effects (font (size 1.5 1.5) (thickness 0.3)) (justify mirror))
   )
-  (gr_text "STM32 CAN <=> USB" (at 175.26 90.17 270) (layer B.SilkS)
-    (effects (font (size 1.5 1.5) (thickness 0.3)) (justify mirror))
-  )
